Commit message: Update rexrov2_base.xacro

File: rexrov2/rexrov2_description/urdf/rexrov2_base.xacro (robot description, xacro)
@@ -20,5 +20,5 @@
   <xacro:property name="visual_mesh_file" value="file://$(find rexrov2_description)/meshes/RexROV2_no_props.dae"/>
   <!-- Mass, see p.28 in Berg2012 -->
-  <xacro:property name="mass" value="1000"/>
+  <xacro:property name="mass" value="5000"/>
 <!--1862.87"/>-->
   <xacro:macro name="rexrov2_base"
